File: presstimer.kicad_pcb (KiCad board)
At the start: 4 copper layers, 93 x 72 mm, 80 parts, among them J1 Screw_Terminal_01x02, J10 Screw_Terminal_01x02, J11 Connector, USB-TYPE-C-16P, J2 Screw_Terminal_01x03, J3 Connector, USB-TYPE-C-16P, J4 Conn_ARM_SWD_TagConnect_TC2030, J5 Conn_01x06_Pin, J6 Conn_01x06_Pin, J8 Screw_Terminal_01x02, J9 Screw_Terminal_01x02, Q10 L8050QLT1G, Q5 Display 2.8" TFT LCD Touch IL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, Q6 AO3401A, Q8 L8050QLT1G, Q9 L8050QLT1G, SW1 SW_Push, SW2 SW_Push, U1 AP7361C-33ER, U2 ESP32-S3-WROOM-1, U3 SFH620A-3X001, U4 SFH620A-3X001, U5 SSR-41FDD, U6 CP2102N-Axx-xQFN28

Commit message: routing finished v0.1.0
Parts:
- added 3V3: TestPoint, TestPoint:TestPoint_Pad_D1.5mm, F.Cu at (132.8, 82.7)
- added 5V: TestPoint, TestPoint:TestPoint_Pad_D1.5mm, F.Cu at (120.6, 82.6)
- added 5V: TestPoint, TestPoint:TestPoint_Pad_D1.5mm, F.Cu at (109.8, 114.7)
- added 5V: TestPoint, TestPoint:TestPoint_Pad_D1.5mm, F.Cu at (110.2, 143.9)
- added GND: TestPoint, TestPoint:TestPoint_Pad_1.5x1.5mm, F.Cu at (113.8, 143.9)
- added GND: TestPoint, TestPoint:TestPoint_Pad_1.5x1.5mm, F.Cu at (129.6, 82.7)
- added GND: TestPoint, TestPoint:TestPoint_Pad_1.5x1.5mm, F.Cu at (112.7, 112.2)
- moved R13 26.4 mm to (178.9, 124.5)
- moved R4 22.7 mm to (178.8, 120.5), turned to -90 degrees
- moved D2 17.8 mm to (183.1, 124.4)
- moved J4 14.7 mm to (172.2, 123.0), turned to 0 degrees
- moved C7 3.60 mm to (110.5, 126.5), turned to 180 degrees
- moved R36 2.22 mm to (176.2, 115.5), turned to -90 degrees
- moved C11 1.82 mm to (123.2, 100.0)
- moved D5 1.82 mm to (119.4, 100.7)
- moved R23 1.40 mm to (109.8, 107.9)
- moved C3 1.30 mm to (136.4, 92.5), turned to 180 degrees
- moved R37 1.20 mm to (178.8, 105.0)
- moved C12 1.14 mm to (178.5, 108.5), turned to 0 degrees
- moved D7 1.09 mm to (116.1, 103.4)
- moved D9 1.09 mm to (114.2, 105.7)
- moved D8 1.03 mm to (185.3, 91.8)
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- renumbered SW1 to BOOT, SW2 to RESET
Connections:
- U1 pad 4: OUT -> Net-(D1-A)
- U2 pad 41: Net-(U2-GND-Pad40) -> GND
- U6 pad 29: Net-(U6-GND-Pad29) -> GND
- U6 pad 3: Net-(U6-GND-Pad29) -> GND
Routing:
- net GND: track 24.1 -> 160.6 mm, vias 0 -> 68
- net +3V3: track 97.7 -> 221.8 mm, vias 0 -> 2
- net SENSE_PRESSURE: track 4.92 -> 68.5 mm, vias 0 -> 2
- net SENSE_RELAIS: track 3.85 -> 50.1 mm, vias 0 -> 4
- net SW_SSR: track 0.66 -> 43.3 mm, vias 0 -> 2
- net UART_RX: track 0.00 -> 40.9 mm, vias 0 -> 2
- net UART_RTS: track 0.00 -> 40.7 mm, vias 0 -> 1
- net UART_TX: track 0.00 -> 37.9 mm, vias 0 -> 2
- net SENSE_VALVE: track 4.94 -> 42.5 mm, vias 0 -> 4
- net CHIP_PU: track 7.72 -> 41.4 mm
- net I2C_INT: track 0.00 -> 30.1 mm, vias 0 -> 1
- net LED_RGB: track 0.00 -> 29.8 mm, vias 0 -> 2
- net D_CS: track 0.00 -> 27.0 mm, vias 0 -> 1
- net UART_CTS: track 0.00 -> 26.6 mm, vias 0 -> 1
- net D_SDI_T_DIN: track 0.00 -> 25.7 mm
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Other:
- outline, holes or cut-outs redrawn
- rule pad_to_mask_clearance: 0 -> 0.05
- board text added: "+"
- board text added: "-"
- board text added: "3V"
- board text added: "5V"
- board text added: "AC"
- board text added: "BL"
- board text added: "CS"
- board text added: "CTS"
- board text added: "DC"
- board text added: "Display"
- board text added: "ESP"
- board text added: "GND"
- board text added: "I2C"
- board text added: "INT"
- board text added: "IO17"
- board text added: "IO7"
- board text added: "L"
- board text added: "N"
- board text added: "PWR"
- board text added: "Pressure"
- board text added: "RST"
- board text added: "RTS"
- board text added: "RX"
- board text added: "Relais"
- board text added: "SCK"
- board text added: "SCL"
- board text added: "SDA"
- board text added: "SDI"
- board text added: "SDO"
- board text added: "SSR"
- board text added: "Sig / IO1"
- board text added: "TC2030"
- board text added: "TX"
- board text added: "T_CLK"
- board text added: "T_CS"
- board text added: "T_DO"
- board text added: "T_IRQ"
- board text added: "UART"
- board text added: "Valve"

Commit message: board finished v1.0
Parts:
- renumbered BOOT to SW1, RESET to SW2, 5V to TP1, 3V3 to TP2, GND to TP3, 5V to TP4, GND to TP5, 5V to TP6, GND to TP7
Connections:
- U2 pad 40: Net-(U2-GND-Pad40) -> GND
Routing:
- net GND: track 160.6 -> 186.8 mm, vias 68 -> 89
- added copper zone on F.Cu, net +3V3
- added copper zone on F.Cu, net +5V
Other:
- outline, holes or cut-outs redrawn
- board text added: "Dualpress Timer"
- board text added: "JLCJLCJLCJLC"
- board text added: "identwear.de"
- board text added: "v1.0 | 2026-06-23"
