File: presstimer.kicad_sch (KiCad schematic)
At the start: 28 parts, among them J1 Screw_Terminal_01x02, SW1 SW_Push, SW2 SW_Push, U1 AP7361C-33ER, U2 ESP32-S3-WROOM-1

Commit message: add: connector heating SSR
Parts:
- removed R1, R2: 4k7, PCM_JLCPCB:R_0603, symbol Device:R
- removed R4: 0, PCM_JLCPCB:R_0805, symbol Device:R
- removed R5, R6: 0, PCM_JLCPCB:R_0603, symbol Device:R
- added Q5: Display 2.8" TFT LCD Touch ILI9431 SPI, Connector_PinHeader_2.54mm:PinHeader_1x14_P2.54mm_Vertical, symbol markus:Display_2.8{dblquote}_TFT_LCD_Touch_ILI9431_SPI
- added Q6: AO3401A, Package_TO_SOT_SMD:SOT-23, symbol PCM_JLCPCB-Transistors:PMOS,AO3401A
- added R16: 100, PCM_JLCPCB:R_0603, symbol Device:R
- added R17: 100k, PCM_JLCPCB:R_0603, symbol Device:R
Connections:
- net +3V3: now also Q5.14 (VCC), Q6.2 (S), R17.1
- net D_BL: now also R16.1
- net D_CS: now also Q5.12 (CS)
- net D_DC: now also Q5.10 (DC)
- net D_RST: now also Q5.11 (RESET)
- net D_SCK_T_CLK: now also Q5.5 (T_CLK), Q5.8 (SCK)
- net D_SDI_T_DIN: now also Q5.3 (T_DIN), Q5.9 (SDI)
- net D_T_CS: now also Q5.4 (T_CS)
- net D_T_DO: now also Q5.2 (T_DO)
- net D_T_IRQ: now also Q5.1 (T_IRQ)
- net GND: now also Q5.13 (GND)
- net LED_RGB: now also R13.1
- net I2C_INT renamed GPIO21
- net I2C_RST renamed GPIO2
- net I2C_SCL renamed GPIO40
- net I2C_SDA renamed GPIO39
- new net: Q6.1 (G), R16.2, R17.2
- new net: Q5.7 (LED), Q6.3 (D)
- no-connect marks 7 -> 8
Other:
- moved on the sheet: C1, C2, D1, F1, J1, R3, TP1, TP2, TP3, U1
