File: usb.kicad_sch (KiCad schematic)
At the start: 35 parts, among them J10 Screw_Terminal_01x02, J12 Conn_01x06_Pin, J2 Screw_Terminal_01x03, J4 Conn_ARM_SWD_TagConnect_TC2030, J5 Conn_01x06_Pin, J6 Conn_01x06_Pin, J8 Screw_Terminal_01x02, J9 Screw_Terminal_01x02, Q10 L8050QLT1G, Q5 Display 2.8" TFT LCD Touch IL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, Q6 AO3401A, U3 SFH620A-3X001, U4 SFH620A-3X001, U5 SSR-41FDD

Commit message: fixed ssr pinout
Parts:
- J2, J8, J9, Q5: now left out of the parts list
- R15, R17, R21, R9: now in the parts list
- U5: footprint markus:SSR-41FDD -> 01_dualpress:SSR-41FDD
Connections:
- net +5V: now also U5.3 (+); no longer U5.1
- net at U5.2: now also J10.2 (Pin_2); no longer Q10.3 (C)
- net at J10.1 (Pin_1): now also U5.1; no longer U5.3
- net at U5.4 (GND): now also Q10.3 (C); no longer J10.2 (Pin_2)
Changed lines of the file:
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@@
 		(body_style 1)
 		(exclude_from_sim no)
-		(in_bom no)
+		(in_bom yes)
 		(on_board yes)
 		(in_pos_files yes)
@@
 		(body_style 1)
 		(exclude_from_sim no)
-		(in_bom yes)
+		(in_bom no)
 		(on_board yes)
 		(in_pos_files yes)
@@
 			)
 		)
-		(property "Footprint" "markus:SSR-41FDD"
+		(property "Footprint" "01_dualpress:SSR-41FDD"
 			(at 223.52 133.35 0)
 			(hide yes)
@@
 		(body_style 1)
 		(exclude_from_sim no)
-		(in_bom no)
+		(in_bom yes)
 		(on_board yes)
 		(in_pos_files yes)
@@
 		(body_style 1)
 		(exclude_from_sim no)
-		(in_bom yes)
+		(in_bom no)
 		(on_board yes)
 		(in_pos_files yes)
@@
 		(body_style 1)
 		(exclude_from_sim no)
-		(in_bom no)
+		(in_bom yes)
 		(on_board yes)
 		(in_pos_files yes)
@@
 		(body_style 1)
 		(exclude_from_sim no)
-		(in_bom yes)
+		(in_bom no)
 		(on_board yes)
 		(in_pos_files yes)
@@
 		(body_style 1)
 		(exclude_from_sim no)
-		(in_bom no)
+		(in_bom yes)
 		(on_board yes)
 		(in_pos_files yes)
@@
 		(body_style 1)
 		(exclude_from_sim no)
-		(in_bom yes)
+		(in_bom no)
 		(on_board yes)
 		(in_pos_files yes)

Commit message: before removal of cp2102
Connections:
- net SENSE_RELAY1: now reaches J8.1 (Pin_1), R22.1
- net SENSE_RELAY2: now reaches J8.2 (Pin_2), U3.2
- net SSR_L: now reaches J10.1 (Pin_1)
- net SSR_L: now also U5.2; no longer U5.1
- net SSR_SW_L: now reaches J10.2 (Pin_2)
- net SSR_SW_L: now also U5.1; no longer U5.2
- net SENSE_SOLENOID2: now reaches J9.2 (Pin_2), U4.2
- net SENSE_SOLENOID1: now reaches J9.1 (Pin_1), R27.1
Other:
- moved on the sheet: J10, J8, J9
Changed lines of the file:
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@@
 	(wire
 		(pts
-			(xy 236.22 130.81) (xy 245.11 130.81)
+			(xy 138.43 173.99) (xy 129.54 173.99)
 		)
 		(stroke
@@
 	(wire
 		(pts
-			(xy 138.43 173.99) (xy 129.54 173.99)
+			(xy 105.41 60.96) (xy 105.41 69.85)
 		)
 		(stroke
@@
 	(wire
 		(pts
-			(xy 105.41 60.96) (xy 105.41 69.85)
+			(xy 369.57 68.58) (xy 369.57 71.12)
 		)
 		(stroke
@@
 	(wire
 		(pts
-			(xy 369.57 68.58) (xy 369.57 71.12)
+			(xy 209.55 83.82) (xy 214.63 83.82)
 		)
 		(stroke
@@
 	(wire
 		(pts
-			(xy 209.55 83.82) (xy 214.63 83.82)
+			(xy 236.22 130.81) (xy 264.16 130.81)
 		)
 		(stroke
@@
 	(wire
 		(pts
-			(xy 245.11 125.73) (xy 236.22 125.73)
+			(xy 242.57 125.73) (xy 236.22 125.73)
 		)
 		(stroke
@@
 	(wire
 		(pts
-			(xy 190.5 41.91) (xy 198.12 41.91)
+			(xy 168.91 41.91) (xy 198.12 41.91)
 		)
 		(stroke
@@
 	(wire
 		(pts
-			(xy 245.11 127) (xy 245.11 125.73)
+			(xy 242.57 127) (xy 242.57 125.73)
+		)
+		(stroke
+			(width 0)
+			(type default)
+		)
+	)
+	(wire
+		(pts
+			(xy 264.16 129.54) (xy 264.16 130.81)
 		)
 		(stroke
@@
 	(wire
 		(pts
-			(xy 190.5 90.17) (xy 198.12 90.17)
+			(xy 173.99 90.17) (xy 198.12 90.17)
 		)
 		(stroke
@@
 	(wire
 		(pts
-			(xy 190.5 87.63) (xy 198.12 87.63)
+			(xy 173.99 87.63) (xy 198.12 87.63)
 		)
 		(stroke
@@
 	(wire
 		(pts
+			(xy 242.57 127) (xy 264.16 127)
+		)
+		(stroke
+			(width 0)
+			(type default)
+		)
+	)
+	(wire
+		(pts
 			(xy 198.12 35.56) (xy 201.93 35.56)
 		)
@@
 	(wire
 		(pts
-			(xy 245.11 130.81) (xy 245.11 129.54)
-		)
-		(stroke
-			(width 0)
-			(type default)
-		)
-	)
-	(wire
-		(pts
 			(xy 46.99 115.57) (xy 46.99 120.65)
 		)
@@
 	(wire
 		(pts
-			(xy 190.5 39.37) (xy 198.12 39.37)
+			(xy 168.91 39.37) (xy 198.12 39.37)
 		)
 		(stroke
@@
 		)
 	)
+	(label "SENSE_RELAY2"
+		(at 191.77 41.91 180)
+		(effects
+			(font
+				(size 1.27 1.27)
+			)
+			(justify right bottom)
+		)
+	)
+	(label "SENSE_SOLENOID1"
+		(at 179.07 87.63 0)
+		(effects
+			(font
+				(size 1.27 1.27)
+			)
+			(justify left bottom)
+		)
+	)
+	(label "SSR_SW_L"
+		(at 257.81 127 180)
+		(effects
+			(font
+				(size 1.27 1.27)
+			)
+			(justify right bottom)
+		)
+	)
+	(label "SENSE_SOLENOID2"
+		(at 179.07 90.17 0)
+		(effects
+			(font
+				(size 1.27 1.27)
+			)
+			(justify left bottom)
+		)
+	)
+	(label "SENSE_RELAY1"
+		(at 191.77 39.37 180)
+		(effects
+			(font
+				(size 1.27 1.27)
+			)
+			(justify right bottom)
+		)
+	)
+	(label "SSR_L"
+		(at 257.81 130.81 180)
+		(effects
+			(font
+				(size 1.27 1.27)
+			)
+			(justify right bottom)
+		)
+	)
 	(global_label "D_BL"
 		(shape input)
@@
 	(symbol
 		(lib_id "Connector:Screw_Terminal_01x02")
-		(at 185.42 39.37 0)
+		(at 163.83 39.37 0)
 		(mirror y)
 		(unit 1)
@@
 		(fields_autoplaced yes)
 		(property "Reference" "J8"
-			(at 185.42 33.02 0)
+			(at 163.83 33.02 0)
 			(show_name no)
 			(do_not_autoplace no)
@@
 		)
 		(property "Value" "Screw_Terminal_01x02"
-			(at 185.42 35.56 0)
+			(at 163.83 35.56 0)
 			(show_name no)
 			(do_not_autoplace no)
@@
 		)
 		(property "Footprint" "markus:DG305-5.0-02P-12-00A(H)"
-			(at 185.42 39.37 0)
+			(at 163.83 39.37 0)
 			(hide yes)
 			(show_name no)
@@
 		)
 		(property "Datasheet" ""
-			(at 185.42 39.37 0)
+			(at 163.83 39.37 0)
 			(hide yes)
 			(show_name no)
@@
 		)
 		(property "Description" "Generic screw terminal, single row, 01x02, script generated (kicad-library-utils/schlib/autogen/connector/)"
-			(at 185.42 39.37 0)
+			(at 163.83 39.37 0)
 			(hide yes)
 			(show_name no)
@@
 		)
 		(property "LCSC" "C5632695"
-			(at 185.42 33.02 0)
+			(at 163.83 33.02 0)
 			(hide yes)
 			(show_name no)
@@
 	(symbol
 		(lib_id "Connector:Screw_Terminal_01x02")
-		(at 250.19 127 0)
+		(at 269.24 129.54 0)
+		(mirror x)
 		(unit 1)
 		(body_style 1)
@@
 		(dnp no)
 		(property "Reference" "J10"
-			(at 250.19 135.89 0)
+			(at 269.24 120.65 0)
 			(show_name no)
 			(do_not_autoplace no)
@@
 		)
 		(property "Value" "Screw_Terminal_01x02"
-			(at 250.19 133.35 0)
+			(at 269.24 123.19 0)
 			(show_name no)
 			(do_not_autoplace no)
@@
 		)
 		(property "Footprint" "markus:DG305-5.0-02P-12-00A(H)"
-			(at 250.19 127 0)
+			(at 269.24 129.54 0)
 			(hide yes)
 			(show_name no)
@@
 		)
 		(property "Datasheet" ""
-			(at 250.19 127 0)
+			(at 269.24 129.54 0)
 			(hide yes)
 			(show_name no)
@@
 		)
 		(property "Description" "Generic screw terminal, single row, 01x02, script generated (kicad-library-utils/schlib/autogen/connector/)"
-			(at 250.19 127 0)
+			(at 269.24 129.54 0)
 			(hide yes)
 			(show_name no)
@@
 		)
 		(property "LCSC" "C5632695"
-			(at 250.19 135.89 0)
+			(at 269.24 120.65 0)
 			(hide yes)
 			(show_name no)
@@
 	(symbol
 		(lib_id "Connector:Screw_Terminal_01x02")
-		(at 185.42 87.63 0)
+		(at 168.91 87.63 0)
 		(mirror y)
 		(unit 1)
@@
 		(fields_autoplaced yes)
 		(property "Reference" "J9"
-			(at 185.42 81.28 0)
+			(at 168.91 81.28 0)
 			(show_name no)
 			(do_not_autoplace no)
@@
 		)
 		(property "Value" "Screw_Terminal_01x02"
-			(at 185.42 83.82 0)
+			(at 168.91 83.82 0)
 			(show_name no)
 			(do_not_autoplace no)
@@
 		)
 		(property "Footprint" "markus:DG305-5.0-02P-12-00A(H)"
-			(at 185.42 87.63 0)
+			(at 168.91 87.63 0)
 			(hide yes)
 			(show_name no)
@@
 		)
 		(property "Datasheet" ""
-			(at 185.42 87.63 0)
+			(at 168.91 87.63 0)
 			(hide yes)
 			(show_name no)
@@
 		)
 		(property "Description" "Generic screw terminal, single row, 01x02, script generated (kicad-library-utils/schlib/autogen/connector/)"
-			(at 185.42 87.63 0)
+			(at 168.91 87.63 0)
 			(hide yes)
 			(show_name no)
@@
 		)
 		(property "LCSC" "C5632695"
-			(at 185.42 81.28 0)
+			(at 168.91 81.28 0)
 			(hide yes)
 			(show_name no)

Commit message: add: connector heating SSR
Parts:
- removed J12, J5: Conn_01x06_Pin, Connector_PinHeader_2.54mm:PinHeader_1x06_P2.54mm_Vertical, symbol Connector:Conn_01x06_Pin
- removed JP4: Jumper_3_Open, Connector:FanPinHeader_1x03_P2.54mm_Vertical, symbol Jumper:Jumper_3_Open
- removed Q5: Display 2.8" TFT LCD Touch ILI9431 SPI, Connector_PinHeader_2.54mm:PinHeader_1x14_P2.54mm_Vertical, symbol markus:Display_2.8{dblquote}_TFT_LCD_Touch_ILI9431_SPI
- removed Q6: AO3401A, Package_TO_SOT_SMD:SOT-23, symbol PCM_JLCPCB-Transistors:PMOS,AO3401A
- removed R16: 100, PCM_JLCPCB:R_0603, symbol Device:R
- removed R17: 100k, PCM_JLCPCB:R_0603, symbol Device:R
- removed R33, R35, R40: 10k, PCM_JLCPCB:R_0603, symbol Device:R
- removed U5: SSR-41FDD, 01_dualpress:SSR-41FDD, symbol SSR-41FDD:SSR-41FDD
- added J5: Screw_Terminal_01x02, markus:DG305-5.0-02P-12-00A(H), symbol Connector:Screw_Terminal_01x02
- added Q1: L8050QLT1G, Package_TO_SOT_SMD:SOT-23, symbol Transistor_BJT:2SC4213
- added R1: 1k, PCM_JLCPCB:R_0603, symbol Device:R
- added TP9: TestPoint, TestPoint:TestPoint_Pad_1.5x1.5mm, symbol Connector:TestPoint
- added U5: SSR-41FDA, markus:SSR-41FDD, symbol SSR-41FDD:SSR-41FDA
- J6: now in the parts list
Connections:
- net +3V3: now also J6.2 (Pin_2); no longer J6.5 (Pin_5)
- net +5V: now also J5.2 (Pin_2), TP9.1, U5.3 (+)
- net GND: now also J6.1 (Pin_1), Q1.2 (E); no longer J6.6 (Pin_6)
- net GPIO14: now also R1.1
- net SSR_L: now also U5.2
- net SSR_SW_L: now also U5.1
- net UART_CTS: now also J6.3 (Pin_3); no longer J6.4 (Pin_4)
- net UART_RTS: now also J6.4 (Pin_4); no longer J6.3 (Pin_3)
- net UART_RX: now also J6.5 (Pin_5); no longer J6.2 (Pin_2)
- net UART_TX: now also J6.6 (Pin_6); no longer J6.1 (Pin_1)
- net at Q10.3 (C): now also U5.4 (GND)
- new net: J5.1 (Pin_1), Q1.3 (C)
- new net: Q1.1 (B), R1.2
- no-connect marks 1 -> 0
Other:
- moved on the sheet: C7, C8, C9, J10, J2, J4, J8, J9, Q10, R10, R15, R21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
